File: KiCAD/Polpoboard_PCB/LED_doubleDigit_sch.kicad_sch (KiCad schematic)
At the start: 6 parts, among them J5 DA15_Plug, U2 74HC595, U3 74HC595, U4 ULN2803A, U5 ULN2803A

Commit message: Minor updates to the PCB
Parts:
- U2, U3: footprint Polpoboard_footprints:74HC595N -> Package_DIP:DIP-16_W7.62mm_Socket_LongPads
- U4, U5: footprint Polpoboard_footprints:ULN2803A -> Package_DIP:DIP-18_W7.62mm_Socket_LongPads
