File: KiCAD/Polpoboard_PCB/Polpoboard_PCB.kicad_sch (KiCad schematic)
At the start: 11 parts, among them J12 +12V IN, J13 +5V external, J2 CONN_LED_MATRIX TeamB, J3 CONN_LED_MATRIX TeamA, J4 +12VDC additional supply, J6 +12VDC additional supply

Commit message: Minor updates to the PCB
Parts:
- added C6: 100nF, symbol Device:C
- added D1: D_Schottky, symbol Device:D_Schottky
- added J10: Conn_01x02_Pin, symbol Connector:Conn_01x02_Pin
- added J8: DE9_Plug_MountingHoles, symbol Connector:DE9_Plug_MountingHoles
- added Q2: IRLZ44N, Package_TO_SOT_THT:TO-220-3_Vertical, symbol Transistor_FET:IRLZ44N
- added R1: R, symbol Device:R
- added U19: TPIC6B595, symbol Polpoboard_parts:TPIC6B595
- J13: value +5V external -> Raspberry Supply
Connections:
- net +12V: now also D1.1 (K), J10.2 (Pin_2), J8.1, J8.6
- net +5V: now also C6.1, U19.2 (VDD), U19.8 (SCL)
- net CLK: now also U19.13 (SCK)
- net GND: now also C6.2, Q2.3 (S), U19.10 (G@1), U19.11 (G@2), U19.19 (G@3), U19.9 (G)
- net SER: now also U19.3 (SER)
- net CS_Halftime: now reaches A?.10 (D7)
- net CS_Halftime: now also U19.12 (RCK)
- net signal_horn: now reaches A?.9 (D6)
- net signal_horn: now also R1.1
- new net: Q2.1 (G), R1.2
- new net: D1.2 (A), J10.1 (Pin_1), Q2.2 (D)
- new net: J8.2, U19.16 (QG)
- new net: J8.3, U19.14 (QE)
- new net: J8.4, U19.6 (QC)
- new net: J8.5, U19.4 (QA)
- new net: J8.7, U19.15 (QF)
- new net: J8.8, U19.7 (QD)
- new net: J8.9, U19.5 (QB)
Other:
- moved on the sheet: J2, J3
