File: KiCAD/Polpoboard_PCB/_autosave-Polpoboard_PCB.kicad_pcb (KiCad board)
At the start: 2 copper layers, 40 parts, among them J11 DA15_Plug, J12 +12V IN, J13 +5V external, J2 CONN_LED_MATRIX TeamB, J3 CONN_LED_MATRIX TeamA, J4 +12VDC additional supply, J5 DA15_Plug, J6 +12VDC additional supply, J7 DA15_Plug, J9 DA15_Plug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

Commit message: Minor updates to the PCB
Parts:
- moved U10 14.3 mm to (119.7, 55.9), turned to 180 degrees
- moved U6 13.7 mm to (119.7, 130.7), turned to 180 degrees
- moved U11 12.9 mm to (119.4, 80.8), turned to 180 degrees
- moved U7 12.9 mm to (119.2, 105.6), turned to 180 degrees
